Commit message: 可以跳一点

File: src/bbot_description/urdf/bbot.urdf.xacro (robot description, xacro)
@@ -2401,6 +2401,6 @@
     <origin xyz="0.3032 0.125 -0.07" rpy="0 0 0" />
     <axis xyz="1 0 0" />
-    <limit lower="-1.57" upper="1.57" effort="150.0" velocity="10" />
-    <dynamics damping="15.0" friction="0.5" />
+    <limit lower="-1.57" upper="1.57" effort="150.0" velocity="30" />
+    <dynamics damping="0.5" friction="0.1" />
   </joint>
   <joint name="link_003_joint" type="revolute">
@@ -2409,6 +2409,6 @@
     <origin xyz="0.072 -0.29348091 -0.06220095" rpy="0 0 0" />
     <axis xyz="1 0 0" />
-    <limit lower="-1.57" upper="1.57" effort="150.0" velocity="10" />
-    <dynamics damping="15.0" friction="0.5" />
+    <limit lower="-1.57" upper="1.57" effort="150.0" velocity="30" />
+    <dynamics damping="0.5" friction="0.1" />
   </joint>
   <joint name="link_004_joint" type="continuous">
@@ -2425,6 +2425,6 @@
     <origin xyz="0.0965 0.125 -0.07" rpy="0 0 0" />
     <axis xyz="1 0 0" />
-    <limit lower="-1.57" upper="1.57" effort="150.0" velocity="10" />
-    <dynamics damping="15.0" friction="0.5" />
+    <limit lower="-1.57" upper="1.57" effort="150.0" velocity="30" />
+    <dynamics damping="0.5" friction="0.1" />
   </joint>
   <joint name="link_006_joint" type="revolute">
@@ -2433,6 +2433,6 @@
     <origin xyz="-0.0667 -0.29348091 -0.06220095" rpy="0 0 0" />
     <axis xyz="1 0 0" />
-    <limit lower="-1.57" upper="1.57" effort="150.0" velocity="10" />
-    <dynamics damping="15.0" friction="0.5" />
+    <limit lower="-1.57" upper="1.57" effort="150.0" velocity="30" />
+    <dynamics damping="0.5" friction="0.1" />
   </joint>
   <joint name="link_007_joint" type="continuous">
@@ -2447,4 +2447,5 @@
     <hardware>
       <plugin>gz_ros2_control/GazeboSimSystem</plugin>
+      <param name="position_proportional_gain">500.0</param>
     </hardware>
     <joint name="link_004_joint">

Commit message: 更改质量与新跳跃控制

File: src/bbot_description/urdf/bbot.urdf.xacro (robot description, xacro)
@@ -1,4 +1,8 @@
 <?xml version='1.0' encoding='utf-8'?>
-<robot name="bbot">
+<robot name="bbot" xmlns:xacro="http://www.ros.org/wiki/xacro">
+  <xacro:arg name="position_proportional_gain" default="0.3" />
+  <xacro:arg name="body_mass" default="9.5" />
+  <xacro:property name="body_mass_value" value="$(arg body_mass)" />
+  <xacro:property name="body_inertia_scale" value="${body_mass_value / 14.0}" />
   <material name="chassis_dark">
     <color rgba="0.18 0.18 0.20 1.0" />
@@ -16,6 +20,11 @@
     <inertial>
       <origin xyz="0.20001846 0.13261282 0.05396677" rpy="0 0 0" />
-      <mass value="14.0" />
-      <inertia ixx="0.159013" ixy="0.000083" ixz="0.000103" iyy="0.269268" iyz="-0.009342" izz="0.233977" />
+      <mass value="${body_mass_value}" />
+      <inertia ixx="${0.159013 * body_inertia_scale}"
+               ixy="${0.000083 * body_inertia_scale}"
+               ixz="${0.000103 * body_inertia_scale}"
+               iyy="${0.269268 * body_inertia_scale}"
+               iyz="${-0.009342 * body_inertia_scale}"
+               izz="${0.233977 * body_inertia_scale}" />
     </inertial>
     <visual name="part_001_visual_1">
@@ -2447,5 +2456,5 @@
     <hardware>
       <plugin>gz_ros2_control/GazeboSimSystem</plugin>
-      <param name="position_proportional_gain">0.1</param>
+      <param name="position_proportional_gain">$(arg position_proportional_gain)</param>
     </hardware>
     <joint name="link_004_joint">
@@ -2540,4 +2549,10 @@
     <plugin filename="ignition-gazebo-imu-system" name="ignition::gazebo::systems::Imu">
     </plugin>
+    <plugin filename="ignition-gazebo-odometry-publisher-system" name="ignition::gazebo::systems::OdometryPublisher">
+      <odom_topic>/model/bbot/odometry</odom_topic>
+      <odom_frame>odom</odom_frame>
+      <robot_base_frame>base_link</robot_base_frame>
+      <dimensions>3</dimensions>
+    </plugin>
   </gazebo>
   <link name="imu_link">

Commit message: 新的自适应算法

File: src/bbot_description/urdf/bbot.urdf.xacro (robot description, xacro)
@@ -2427,5 +2427,5 @@
     <axis xyz="1 0 0" />
     <limit effort="50.0" velocity="30" />
-    <dynamics damping="0.1" friction="0.05" />
+    <dynamics damping="0.1" friction="0.0" />
   </joint>
   <joint name="link_005_joint" type="revolute">
@@ -2451,5 +2451,5 @@
     <axis xyz="1 0 0" />
     <limit effort="50.0" velocity="30" />
-    <dynamics damping="0.1" friction="0.05" />
+    <dynamics damping="0.1" friction="0.0" />
   </joint>
   <ros2_control name="bbot_hardware_interface" type="system">

Commit message: 加入载荷实验

File: src/bbot_description/urdf/bbot.urdf.xacro (robot description, xacro)
@@ -2660,3 +2660,60 @@
     </visual>
   </gazebo>
+  <!-- ==================== Payload Options ==================== -->
+  <xacro:arg name="payload_mass" default="0.0" />
+  <xacro:arg name="payload_x" default="0.200" />
+  <xacro:arg name="payload_y_offset" default="0.0" />
+  <xacro:arg name="payload_z" default="0.170" />
+  <xacro:arg name="payload_size_x" default="0.12" />
+  <xacro:arg name="payload_size_y" default="0.08" />
+  <xacro:arg name="payload_size_z" default="0.02" />
+  <xacro:property name="p_mass" value="${float('$(arg payload_mass)')}" />
+  <xacro:property name="p_x" value="${float('$(arg payload_x)')}" />
+  <xacro:property name="p_y_off" value="${float('$(arg payload_y_offset)')}" />
+  <xacro:property name="p_z" value="${float('$(arg payload_z)')}" />
+  <xacro:property name="p_lx" value="${float('$(arg payload_size_x)')}" />
+  <xacro:property name="p_ly" value="${float('$(arg payload_size_y)')}" />
+  <xacro:property name="p_lz" value="${float('$(arg payload_size_z)')}" />
+  <xacro:if value="${p_mass > 1e-4}">
+    <link name="payload_link">
+      <inertial>
+        <origin xyz="0 0 0" rpy="0 0 0" />
+        <mass value="${p_mass}" />
+        <inertia ixx="${p_mass * (p_ly * p_ly + p_lz * p_lz) / 12.0}"
+                 ixy="0.0" ixz="0.0"
+                 iyy="${p_mass * (p_lx * p_lx + p_lz * p_lz) / 12.0}"
+                 iyz="0.0"
+                 izz="${p_mass * (p_lx * p_lx + p_ly * p_ly) / 12.0}" />
+      </inertial>
+      <visual>
+        <origin xyz="0 0 0" rpy="0 0 0" />
+        <geometry>
+          <box size="${p_lx} ${p_ly} ${p_lz}" />
+        </geometry>
+        <material name="payload_orange">
+          <color rgba="0.92 0.45 0.10 1.0" />
+        </material>
+      </visual>
+      <collision>
+        <origin xyz="0 0 0" rpy="0 0 0" />
+        <geometry>
+          <box size="${p_lx} ${p_ly} ${p_lz}" />
+        </geometry>
+      </collision>
+    </link>
+    <joint name="payload_joint" type="fixed">
+      <parent link="base_link" />
+      <child link="payload_link" />
+      <origin xyz="${p_x} ${0.125 + p_y_off} ${p_z}" rpy="0 0 0" />
+    </joint>
+    <gazebo reference="payload_link">
+      <visual>
+        <material>
+          <ambient>0.92 0.45 0.10 1.0</ambient>
+          <diffuse>0.92 0.45 0.10 1.0</diffuse>
+          <specular>0.5 0.5 0.5 1.0</specular>
+        </material>
+      </visual>
+    </gazebo>
+  </xacro:if>
 </robot>

Commit message: Backup source, flat jump reports, and handoff plan

File: src/bbot_description/urdf/bbot.urdf.xacro (robot description, xacro)
@@ -2548,8 +2548,22 @@
     <mu1>1.0</mu1>
     <mu2>1.0</mu2>
+    <sensor name="left_wheel_contact" type="contact">
+      <always_on>true</always_on>
+      <update_rate>100</update_rate>
+      <contact>
+        <collision>link_004_collision_collision</collision>
+      </contact>
+    </sensor>
   </gazebo>
   <gazebo reference="link_007">
     <mu1>1.0</mu1>
     <mu2>1.0</mu2>
+    <sensor name="right_wheel_contact" type="contact">
+      <always_on>true</always_on>
+      <update_rate>100</update_rate>
+      <contact>
+        <collision>link_007_collision_collision</collision>
+      </contact>
+    </sensor>
   </gazebo>
   <gazebo>
